File: cartridge-pcb/Cartridge-PCB.kicad_sch (KiCad schematic)
At the start: 13 parts, among them J1 Conn_01x06_Pin, J2 Conn_01x03_Socket, J3 Conn_01x03_Pin, SW1 SW_DIP_x03

Commit message: minor fixes
Parts:
- removed J2: Conn_01x03_Socket, Connector_Wire:SolderWire-0.5sqmm_1x03_P4.6mm_D0.9mm_OD2.1mm, symbol Connector:Conn_01x03_Socket
- U1: value (none) -> Teensy40
Changed lines of the file:
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@@
-	)
-	(junction
-		(at 204.47 97.79)
-		(diameter 0)
-		(color 0 0 0 0)
 	)
 	(junction
@@
 	)
 	(junction
-		(at 207.01 92.71)
-		(diameter 0)
-		(color 0 0 0 0)
-	)
-	(junction
 		(at 184.15 100.33)
-		(diameter 0)
-		(color 0 0 0 0)
-	)
-	(junction
-		(at 205.74 95.25)
 		(diameter 0)
 		(color 0 0 0 0)
@@
 	(wire
 		(pts
-			(xy 210.82 106.68) (xy 204.47 106.68)
-		)
-		(stroke
-			(width 0)
-			(type default)
-		)
-	)
-	(wire
-		(pts
 			(xy 144.78 99.06) (xy 143.51 99.06)
 		)
@@
 	(wire
 		(pts
-			(xy 204.47 106.68) (xy 204.47 97.79)
-		)
-		(stroke
-			(width 0)
-			(type default)
-		)
-	)
-	(wire
-		(pts
 			(xy 111.76 44.45) (xy 115.57 44.45)
 		)
@@
 	(wire
 		(pts
-			(xy 210.82 104.14) (xy 205.74 104.14)
-		)
-		(stroke
-			(width 0)
-			(type default)
-		)
-	)
-	(wire
-		(pts
-			(xy 205.74 95.25) (xy 201.93 95.25)
-		)
-		(stroke
-			(width 0)
-			(type default)
-		)
-	)
-	(wire
-		(pts
 			(xy 208.28 77.47) (xy 199.39 77.47)
 		)
@@
 	(wire
 		(pts
-			(xy 210.82 95.25) (xy 205.74 95.25)
+			(xy 201.93 95.25) (xy 210.82 95.25)
 		)
 		(stroke
@@
 	(wire
 		(pts
-			(xy 205.74 104.14) (xy 205.74 95.25)
-		)
-		(stroke
-			(width 0)
-			(type default)
-		)
-	)
-	(wire
-		(pts
 			(xy 85.09 96.52) (xy 95.25 96.52)
 		)
@@
 	(wire
 		(pts
-			(xy 207.01 92.71) (xy 210.82 92.71)
-		)
-		(stroke
-			(width 0)
-			(type default)
-		)
-	)
-	(wire
-		(pts
-			(xy 210.82 101.6) (xy 207.01 101.6)
-		)
-		(stroke
-			(width 0)
-			(type default)
-		)
-	)
-	(wire
-		(pts
 			(xy 77.47 80.01) (xy 77.47 82.55)
 		)
@@
 	(wire
 		(pts
-			(xy 207.01 101.6) (xy 207.01 92.71)
-		)
-		(stroke
-			(width 0)
-			(type default)
-		)
-	)
-	(wire
-		(pts
 			(xy 77.47 77.47) (xy 74.93 77.47)
 		)
@@
 	(wire
 		(pts
-			(xy 204.47 97.79) (xy 210.82 97.79)
+			(xy 184.15 97.79) (xy 210.82 97.79)
 		)
 		(stroke
@@
 	(wire
 		(pts
-			(xy 193.04 92.71) (xy 207.01 92.71)
+			(xy 193.04 92.71) (xy 210.82 92.71)
 		)
 		(stroke
@@
 		(pts
 			(xy 85.09 93.98) (xy 95.25 93.98)
-		)
-		(stroke
-			(width 0)
-			(type default)
-		)
-	)
-	(wire
-		(pts
-			(xy 184.15 97.79) (xy 204.47 97.79)
 		)
 		(stroke
@@
 	(symbol
 		(lib_id "Connector:Conn_01x03_Pin")
-		(at 215.9 104.14 180)
+		(at 215.9 95.25 180)
 		(unit 1)
 		(body_style 1)
@@
 		(fields_autoplaced yes)
 		(property "Reference" "J3"
-			(at 217.17 102.8699 0)
+			(at 217.17 93.9799 0)
 			(show_name no)
 			(do_not_autoplace no)
@@
 		)
 		(property "Value" "Conn_01x03_Pin"
-			(at 217.17 105.4099 0)
+			(at 217.17 96.5199 0)
 			(show_name no)
 			(do_not_autoplace no)
@@
 		)
 		(property "Footprint" "Connector_JST:JST_XH_B3B-XH-A_1x03_P2.50mm_Vertical"
-			(at 215.9 104.14 0)
+			(at 215.9 95.25 0)
 			(hide yes)
 			(show_name no)
@@
 		)
 		(property "Datasheet" ""
-			(at 215.9 104.14 0)
+			(at 215.9 95.25 0)
 			(hide yes)
 			(show_name no)
@@
 		)
 		(property "Description" "Generic connector, single row, 01x03, script generated"
-			(at 215.9 104.14 0)
+			(at 215.9 95.25 0)
 			(hide yes)
 			(show_name no)
@@
 			)
 		)
-		(property "Value" ""
+		(property "Value" "Teensy40"
 			(at 119.38 64.77 0)
 			(show_name no)
@@
 					(unit 1)
 				)
-			)
-		)
-	)
-	(symbol
-		(lib_id "Connector:Conn_01x03_Socket")
-		(at 215.9 95.25 0)
-		(unit 1)
-		(body_style 1)
-		(exclude_from_sim no)
-		(in_bom yes)
-		(on_board yes)
-		(in_pos_files yes)
-		(dnp no)
-		(fields_autoplaced yes)
-		(property "Reference" "J2"
-			(at 217.17 93.9799 0)
-			(show_name no)
-			(do_not_autoplace no)
-			(effects
-				(font
-					(size 1.27 1.27)
-				)
-				(justify left)
-			)
-		)
-		(property "Value" "Conn_01x03_Socket"
-			(at 217.17 96.5199 0)
-			(show_name no)
-			(do_not_autoplace no)
-			(effects
-				(font
-					(size 1.27 1.27)
-				)
-				(justify left)
-			)
-		)
-		(property "Footprint" "Connector_Wire:SolderWire-0.5sqmm_1x03_P4.6mm_D0.9mm_OD2.1mm"
-			(at 215.9 95.25 0)
-			(hide yes)
-			(show_name no)
-			(do_not_autoplace no)
-			(effects
-				(font
-					(size 1.27 1.27)
-				)
-			)
-		)
-		(property "Datasheet" ""
-			(at 215.9 95.25 0)
-			(hide yes)
-			(show_name no)
-			(do_not_autoplace no)
-			(effects
-				(font
-					(size 1.27 1.27)
-				)
-			)
-		)
-		(property "Description" "Generic connector, single row, 01x03, script generated"
-			(at 215.9 95.25 0)
-			(hide yes)
-			(show_name no)
-			(do_not_autoplace no)
-			(effects
-				(font
-					(size 1.27 1.27)
-				)
-			)
-		)
-		(pin "2"
-		)
-		(pin "3"
-		)
-		(pin "1"
-		)
-		(instances
-			(project "Cartridge-PCB"
-				(path "/d783fe36-1ab4-412e-a370-8ddb0a7d9565"
-					(reference "J2")
-					(unit 1)
-				)
